Commit message: replace adam_pick gripper with hand_pw
Ultraworked with [Sisyphus](https://github.com/code-yeongyu/oh-my-openagent)

Co-authored-by: Sisyphus <clio-agent@sisyphuslabs.ai>

File: adam_pick/adam_pro_omnipicker.urdf (robot description, URDF)
Before this commit: robot adam_pro_omnipicker, 57 links, 56 joints
Links:
- removed link op_l_base_link
- removed link op_l_hand_narrow1_Link
- removed link op_l_hand_narrow2_Link
- removed link op_l_hand_narrow3_Link
- removed link op_l_hand_narrow4_Link
- removed link op_l_hand_narrow_loop_Link
- removed link op_l_hand_wide1_Link
- removed link op_l_hand_wide2_Link
- removed link op_l_hand_wide3_Link
- removed link op_l_hand_wide4_Link
- removed link op_l_hand_wide_loop_Link
- removed link op_r_base_link
- removed link op_r_hand_narrow1_Link
- removed link op_r_hand_narrow2_Link
- removed link op_r_hand_narrow3_Link
- removed link op_r_hand_narrow4_Link
- removed link op_r_hand_narrow_loop_Link
- removed link op_r_hand_wide1_Link
- removed link op_r_hand_wide2_Link
- removed link op_r_hand_wide3_Link
- removed link op_r_hand_wide4_Link
- removed link op_r_hand_wide_loop_Link
- added link gripper_l_base_link, mass 1.3757592; collision mesh filename=meshes_stl_0.25/wuliao_Collision_01.STL; collision mesh filename=meshes_stl_0.25/wuliao_Collision_02.STL
- added link gripper_l_center_link
- added link gripper_l_inner_link1, mass 0.0379014
- added link gripper_l_outer_link1, mass 0.0366645
- added link gripper_r_base_link, mass 1.3757592; visual mesh filename=meshes_stl_0.25/base_link.STL
- added link gripper_r_center_link
- added link gripper_r_inner_link1, mass 0.0379014
- added link gripper_r_outer_link1, mass 0.0366645
- added link workpiece_r
- added link workpiece_r_collision_01
- added link workpiece_r_collision_01_visual; collision mesh filename=meshes_stl_0.25/wuliao_Collision_01.STL
- added link workpiece_r_collision_02
- added link workpiece_r_collision_02_visual; collision mesh filename=meshes_stl_0.25/wuliao_Collision_02.STL
- added link workpiece_r_collision_03
- added link workpiece_r_collision_03_visual; collision mesh filename=meshes_stl_0.25/wuliao_Collision_03.STL
- added link workpiece_r_collision_04
- added link workpiece_r_collision_04_visual; collision mesh filename=meshes_stl_0.25/wuliao_Collision_04.STL
- added link workpiece_r_collision_05
- added link workpiece_r_collision_05_visual; collision mesh filename=meshes_stl_0.25/wuliao_Collision_05.STL
- added link workpiece_r_collision_06
- added link workpiece_r_collision_06_visual; collision mesh filename=meshes_stl_0.25/wuliao_Collision_06.STL
- added link workpiece_r_collision_07
- added link workpiece_r_collision_07_visual; collision mesh filename=meshes_stl_0.25/wuliao_Collision_07.STL
- added link workpiece_r_collision_08
- added link workpiece_r_collision_08_visual; collision mesh filename=meshes_stl_0.25/wuliao_Collision_08.STL
- added link workpiece_r_collision_09
- added link workpiece_r_collision_09_visual; collision mesh filename=meshes_stl_0.25/wuliao_Collision_09.STL
- added link workpiece_r_collision_10
- added link workpiece_r_collision_10_visual; collision mesh filename=meshes_stl_0.25/wuliao_Collision_10.STL
- added link workpiece_r_collision_11
- added link workpiece_r_collision_11_visual; collision mesh filename=meshes_stl_0.25/wuliao_Collision_11.STL
Joints:
- removed joint left_gripper_joint
- removed joint op_l_base_link_joint
- removed joint op_l_hand_narrow2_joint
- removed joint op_l_hand_narrow3_joint
- removed joint op_l_hand_narrow4_joint
- removed joint op_l_hand_narrow_loop_joint
- removed joint op_l_hand_wide1_joint
- removed joint op_l_hand_wide2_joint
- removed joint op_l_hand_wide3_joint
- removed joint op_l_hand_wide4_joint
- removed joint op_l_hand_wide_loop_joint
- removed joint op_r_base_link_joint
- removed joint op_r_hand_narrow2_joint
- removed joint op_r_hand_narrow3_joint
- removed joint op_r_hand_narrow4_joint
- removed joint op_r_hand_narrow_loop_joint
- removed joint op_r_hand_wide1_joint
- removed joint op_r_hand_wide2_joint
- removed joint op_r_hand_wide3_joint
- removed joint op_r_hand_wide4_joint
- removed joint op_r_hand_wide_loop_joint
- removed joint right_gripper_joint
- added joint gripper_l_base_link_joint: type fixed, parent wristRollLeft, child gripper_l_base_link, origin xyz=0.095 0 0 rpy=-1.5707963267948966 0 -1.5707963267948966
- added joint gripper_l_center_joint: type fixed, parent gripper_l_base_link, child gripper_l_center_link, origin xyz=0 0 0.1 rpy=0 0 -1.5707969456925137
- added joint gripper_r_base_link_joint: type fixed, parent wristRollRight, child gripper_r_base_link, origin xyz=0.095 0 0 rpy=-1.5707963267948966 0 -1.5707963267948966
- added joint gripper_r_center_joint: type fixed, parent gripper_r_base_link, child gripper_r_center_link, origin xyz=0 0 0.1 rpy=0 0 -1.5707969456925137
- added joint idx31_gripper_l_inner_joint1: type prismatic, parent gripper_l_base_link, child gripper_l_inner_link1, origin xyz=-0.0265 0.0134 0.098 rpy=0 0 -1.5707969456925137, axis 0 1 0, limit lower=0 upper=0.024 effort=500 velocity=1
- added joint idx41_gripper_l_outer_joint1: type prismatic, parent gripper_l_base_link, child gripper_l_outer_link1, origin xyz=0.0265 -0.0134 0.098 rpy=0 0 1.5707969456925137, axis 0 1 0, limit lower=0 upper=0.024 effort=500 velocity=1, mimic joint=idx31_gripper_l_inner_joint1 multiplier=1 offset=0
- added joint idx71_gripper_r_inner_joint1: type prismatic, parent gripper_r_base_link, child gripper_r_inner_link1, origin xyz=-0.0265 0.0134 0.098 rpy=0 0 -1.5707969456925137, axis 0 1 0, limit lower=0 upper=0.024 effort=500 velocity=1
- added joint idx81_gripper_r_outer_joint1: type prismatic, parent gripper_r_base_link, child gripper_r_outer_link1, origin xyz=0.0265 -0.0134 0.098 rpy=0 0 1.5707969456925137, axis 0 1 0, limit lower=0 upper=0.024 effort=500 velocity=1, mimic joint=idx71_gripper_r_inner_joint1 multiplier=1 offset=0
- added joint workpiece_r_collision_01_joint: type fixed, parent workpiece_r, child workpiece_r_collision_01, origin xyz=0 0 0 rpy=0 0 0
- added joint workpiece_r_collision_01_visual_joint: type fixed, parent workpiece_r_collision_01, child workpiece_r_collision_01_visual, origin xyz=0 0 0 rpy=0 0 0
- added joint workpiece_r_collision_02_joint: type fixed, parent workpiece_r, child workpiece_r_collision_02, origin xyz=0 0 0 rpy=0 0 0
- added joint workpiece_r_collision_02_visual_joint: type fixed, parent workpiece_r_collision_02, child workpiece_r_collision_02_visual, origin xyz=0 0 0 rpy=0 0 0
- added joint workpiece_r_collision_03_joint: type fixed, parent workpiece_r, child workpiece_r_collision_03, origin xyz=0 0 0 rpy=0 0 0
- added joint workpiece_r_collision_03_visual_joint: type fixed, parent workpiece_r_collision_03, child workpiece_r_collision_03_visual, origin xyz=0 0 0 rpy=0 0 0
- added joint workpiece_r_collision_04_joint: type fixed, parent workpiece_r, child workpiece_r_collision_04, origin xyz=0 0 0 rpy=0 0 0
- added joint workpiece_r_collision_04_visual_joint: type fixed, parent workpiece_r_collision_04, child workpiece_r_collision_04_visual, origin xyz=0 0 0 rpy=0 0 0
- added joint workpiece_r_collision_05_joint: type fixed, parent workpiece_r, child workpiece_r_collision_05, origin xyz=0 0 0 rpy=0 0 0
- added joint workpiece_r_collision_05_visual_joint: type fixed, parent workpiece_r_collision_05, child workpiece_r_collision_05_visual, origin xyz=0 0 0 rpy=0 0 0
- added joint workpiece_r_collision_06_joint: type fixed, parent workpiece_r, child workpiece_r_collision_06, origin xyz=0 0 0 rpy=0 0 0
- added joint workpiece_r_collision_06_visual_joint: type fixed, parent workpiece_r_collision_06, child workpiece_r_collision_06_visual, origin xyz=0 0 0 rpy=0 0 0
- added joint workpiece_r_collision_07_joint: type fixed, parent workpiece_r, child workpiece_r_collision_07, origin xyz=0 0 0 rpy=0 0 0
- added joint workpiece_r_collision_07_visual_joint: type fixed, parent workpiece_r_collision_07, child workpiece_r_collision_07_visual, origin xyz=0 0 0 rpy=0 0 0
- added joint workpiece_r_collision_08_joint: type fixed, parent workpiece_r, child workpiece_r_collision_08, origin xyz=0 0 0 rpy=0 0 0
- added joint workpiece_r_collision_08_visual_joint: type fixed, parent workpiece_r_collision_08, child workpiece_r_collision_08_visual, origin xyz=0 0 0 rpy=0 0 0
- added joint workpiece_r_collision_09_joint: type fixed, parent workpiece_r, child workpiece_r_collision_09, origin xyz=0 0 0 rpy=0 0 0
- added joint workpiece_r_collision_09_visual_joint: type fixed, parent workpiece_r_collision_09, child workpiece_r_collision_09_visual, origin xyz=0 0 0 rpy=0 0 0
- added joint workpiece_r_collision_10_joint: type fixed, parent workpiece_r, child workpiece_r_collision_10, origin xyz=0 0 0 rpy=0 0 0
- added joint workpiece_r_collision_10_visual_joint: type fixed, parent workpiece_r_collision_10, child workpiece_r_collision_10_visual, origin xyz=0 0 0 rpy=0 0 0
- added joint workpiece_r_collision_11_joint: type fixed, parent workpiece_r, child workpiece_r_collision_11, origin xyz=0 0 0 rpy=0 0 0
- added joint workpiece_r_collision_11_visual_joint: type fixed, parent workpiece_r_collision_11, child workpiece_r_collision_11_visual, origin xyz=0 0 0 rpy=0 0 0
- added joint workpiece_r_joint: type fixed, parent gripper_r_base_link, child workpiece_r, origin xyz=0 0 0 rpy=0 0 0

Commit message: replace adam_pick gripper with G1 omnipicker source
Ultraworked with [Sisyphus](https://github.com/code-yeongyu/oh-my-openagent)

Co-authored-by: Sisyphus <clio-agent@sisyphuslabs.ai>

File: adam_pick/adam_pro_omnipicker.urdf (robot description, URDF)
Before this commit: robot adam_pro_omnipicker, 66 links, 65 joints
Links:
- removed link workpiece_r
- removed link workpiece_r_collision_01
- removed link workpiece_r_collision_01_visual
- removed link workpiece_r_collision_02
- removed link workpiece_r_collision_02_visual
- removed link workpiece_r_collision_03
- removed link workpiece_r_collision_03_visual
- removed link workpiece_r_collision_04
- removed link workpiece_r_collision_04_visual
- removed link workpiece_r_collision_05
- removed link workpiece_r_collision_05_visual
- removed link workpiece_r_collision_06
- removed link workpiece_r_collision_06_visual
- removed link workpiece_r_collision_07
- removed link workpiece_r_collision_07_visual
- removed link workpiece_r_collision_08
- removed link workpiece_r_collision_08_visual
- removed link workpiece_r_collision_09
- removed link workpiece_r_collision_09_visual
- removed link workpiece_r_collision_10
- removed link workpiece_r_collision_10_visual
- removed link workpiece_r_collision_11
- removed link workpiece_r_collision_11_visual
- added link gripper_l_inner_link2, mass 0.022591; collision mesh filename=package://genie_robot_description/meshes/omnipicker/inner_l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; visual mesh filename=package://genie_robot_description/meshes/omnipicker/inner_l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
- added link gripper_l_inner_link3, mass 0.0040132; collision mesh filename=package://genie_robot_description/meshes/omnipicker/inner_l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; visual mesh filename=package://genie_robot_description/meshes/omnipicker/inner_l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
- added link gripper_l_inner_link4, mass 0.018029; collision mesh filename=package://genie_robot_description/meshes/omnipicker/inner_l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; visual mesh filename=package://genie_robot_description/meshes/omnipicker/inner_l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
- added link gripper_l_outer_link2, mass 0.025142; collision mesh filename=package://genie_robot_description/meshes/omnipicker/outer_l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; visual mesh filename=package://genie_robot_description/meshes/omnipicker/outer_l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
- added link gripper_l_outer_link3, mass 0.0040132; collision mesh filename=package://genie_robot_description/meshes/omnipicker/outer_l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; visual mesh filename=package://genie_robot_description/meshes/omnipicker/outer_l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
- added link gripper_l_outer_link4, mass 0.035835; collision mesh filename=package://genie_robot_description/meshes/omnipicker/outer_l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; visual mesh filename=package://genie_robot_description/meshes/omnipicker/outer_l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
- added link gripper_r_inner_link2, mass 0.022591; collision mesh filename=package://genie_robot_description/meshes/omnipicker/inner_l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; visual mesh filename=package://genie_robot_description/meshes/omnipicker/inner_l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
- added link gripper_r_inner_link3, mass 0.0040132; collision mesh filename=package://genie_robot_description/meshes/omnipicker/inner_l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; visual mesh filename=package://genie_robot_description/meshes/omnipicker/inner_l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
- added link gripper_r_inner_link4, mass 0.018029; collision mesh filename=package://genie_robot_description/meshes/omnipicker/inner_l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; visual mesh filename=package://genie_robot_description/meshes/omnipicker/inner_l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
- added link gripper_r_outer_link2, mass 0.025142; collision mesh filename=package://genie_robot_description/meshes/omnipicker/outer_l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; visual mesh filename=package://genie_robot_description/meshes/omnipicker/outer_l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
- added link gripper_r_outer_link3, mass 0.0040132; collision mesh filename=package://genie_robot_description/meshes/omnipicker/outer_l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; visual mesh filename=package://genie_robot_description/meshes/omnipicker/outer_l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
- added link gripper_r_outer_link4, mass 0.035835; collision mesh filename=package://genie_robot_description/meshes/omnipicker/outer_l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; visual mesh filename=package://genie_robot_description/meshes/omnipicker/outer_l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
- link gripper_l_base_link: mass 1.3757592 -> 0.23588; geometry collision mesh filename=package://genie_robot_description/meshes/omnipicker/gripper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; visual mesh filename=package://genie_robot_description/meshes/omnipicker/gripper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
- link gripper_l_inner_link1: mass 0.0379014 -> 0.025428; geometry collision mesh filename=package://genie_robot_description/meshes/omnipicker/inner_l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; visual mesh filename=package://genie_robot_description/meshes/omnipicker/inner_l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
- link gripper_l_outer_link1: mass 0.0366645 -> 0.025428; geometry collision mesh filename=package://genie_robot_description/meshes/omnipicker/outer_l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; visual mesh filename=package://genie_robot_description/meshes/omnipicker/outer_l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
- link gripper_r_base_link: mass 1.3757592 -> 0.23588; geometry collision mesh filename=package://genie_robot_description/meshes/omnipicker/gripper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; visual mesh filename=package://genie_robot_description/meshes/omnipicker/gripper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
- link gripper_r_inner_link1: mass 0.0379014 -> 0.025428; geometry collision mesh filename=package://genie_robot_description/meshes/omnipicker/inner_l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; visual mesh filename=package://genie_robot_description/meshes/omnipicker/inner_l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
- link gripper_r_outer_link1: mass 0.0366645 -> 0.025428; geometry collision mesh filename=package://genie_robot_description/meshes/omnipicker/outer_l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; visual mesh filename=package://genie_robot_description/meshes/omnipicker/outer_l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
Joints:
- removed joint gripper_l_base_link_joint
- removed joint gripper_l_center_joint
- removed joint gripper_r_base_link_joint
- removed joint gripper_r_center_joint
- removed joint workpiece_r_collision_01_joint
- removed joint workpiece_r_collision_01_visual_joint
- removed joint workpiece_r_collision_02_joint
- removed joint workpiece_r_collision_02_visual_joint
- removed joint workpiece_r_collision_03_joint
- removed joint workpiece_r_collision_03_visual_joint
- removed joint workpiece_r_collision_04_joint
- removed joint workpiece_r_collision_04_visual_joint
- removed joint workpiece_r_collision_05_joint
- removed joint workpiece_r_collision_05_visual_joint
- removed joint workpiece_r_collision_06_joint
- removed joint workpiece_r_collision_06_visual_joint
- removed joint workpiece_r_collision_07_joint
- removed joint workpiece_r_collision_07_visual_joint
- removed joint workpiece_r_collision_08_joint
- removed joint workpiece_r_collision_08_visual_joint
- removed joint workpiece_r_collision_09_joint
- removed joint workpiece_r_collision_09_visual_joint
- removed joint workpiece_r_collision_10_joint
- removed joint workpiece_r_collision_10_visual_joint
- removed joint workpiece_r_collision_11_joint
- removed joint workpiece_r_collision_11_visual_joint
- removed joint workpiece_r_joint
- added joint idx32_gripper_l_inner_joint3: type revolute, parent gripper_l_inner_link1, child gripper_l_inner_link3, origin xyz=0.030852 0.018551 0 rpy=0 0 0, axis 0 0 -1, limit lower=-2 upper=2 effort=10 velocity=10
- added joint idx33_gripper_l_inner_joint4: type revolute, parent gripper_l_inner_link3, child gripper_l_inner_link4, origin xyz=0.018118 -0.01574 0 rpy=0 0 0, axis 0 0 1, limit lower=-2 upper=2 effort=10 velocity=10
- added joint idx39_gripper_l_inner_joint2: type revolute, parent gripper_l_base_link, child gripper_l_inner_link2, origin xyz=0 -0.021633 0.07387 rpy=-2.9951 -1.5707963267948966 -0.15964, axis 0 0 -1, limit lower=-2 upper=2 effort=10 velocity=10
- added joint idx42_gripper_l_outer_joint3: type revolute, parent gripper_l_outer_link1, child gripper_l_outer_link3, origin xyz=0.030852 -0.018551 0 rpy=0 0 0, axis 0 0 -1, limit lower=-2 upper=2 effort=10 velocity=10
- added joint idx43_gripper_l_outer_joint4: type revolute, parent gripper_l_outer_link3, child gripper_l_outer_link4, origin xyz=0.018118 0.01574 0 rpy=0 0 0, axis 0 0 -1, limit lower=-2 upper=2 effort=10 velocity=10
- added joint idx49_gripper_l_outer_joint2: type revolute, parent gripper_l_base_link, child gripper_l_outer_link2, origin xyz=0 0.021633 0.07387 rpy=-2.9951 -1.5707963267948966 -0.15964, axis 0 0 -1, limit lower=-2 upper=2 effort=10 velocity=10
- added joint idx51_ee_l_joint: type fixed, parent arm_l_link7, child gripper_l_base_link, origin xyz=0 0 0.0061 rpy=0 0 1.5707963267948966, axis 0 0 0
- added joint idx52_gripper_l_center_joint: type fixed, parent gripper_l_base_link, child gripper_l_center_link, origin xyz=0.0 0.0 0.14308 rpy=0 0 -1.5707963267948966
- added joint idx72_gripper_r_inner_joint3: type revolute, parent gripper_r_inner_link1, child gripper_r_inner_link3, origin xyz=0.030852 0.018551 0 rpy=0 0 0, axis 0 0 -1, limit lower=-2 upper=2 effort=10 velocity=10
- added joint idx73_gripper_r_inner_joint4: type revolute, parent gripper_r_inner_link3, child gripper_r_inner_link4, origin xyz=0.018118 -0.01574 0 rpy=0 0 0, axis 0 0 1, limit lower=-2 upper=2 effort=10 velocity=10
- added joint idx79_gripper_r_inner_joint2: type revolute, parent gripper_r_base_link, child gripper_r_inner_link2, origin xyz=0 -0.021633 0.07387 rpy=-2.9951 -1.5707963267948966 -0.15964, axis 0 0 -1, limit lower=-2 upper=2 effort=10 velocity=10
- added joint idx82_gripper_r_outer_joint3: type revolute, parent gripper_r_outer_link1, child gripper_r_outer_link3, origin xyz=0.030852 -0.018551 0 rpy=0 0 0, axis 0 0 -1, limit lower=-2 upper=2 effort=10 velocity=10
- added joint idx83_gripper_r_outer_joint4: type revolute, parent gripper_r_outer_link3, child gripper_r_outer_link4, origin xyz=0.018118 0.01574 0 rpy=0 0 0, axis 0 0 -1, limit lower=-2 upper=2 effort=10 velocity=10
- added joint idx89_gripper_r_outer_joint2: type revolute, parent gripper_r_base_link, child gripper_r_outer_link2, origin xyz=0 0.021633 0.07387 rpy=-2.9951 -1.5707963267948966 -0.15964, axis 0 0 -1, limit lower=-2 upper=2 effort=10 velocity=10
- added joint idx91_ee_r_joint: type fixed, parent arm_r_link7, child gripper_r_base_link, origin xyz=0 0 0 rpy=0 0 -1.5707963267948966, axis 0 0 0
- added joint idx92_gripper_r_center_joint: type fixed, parent gripper_r_base_link, child gripper_r_center_link, origin xyz=0.0 0.0 0.14308 rpy=0 0 -1.5707963267948966
- joint idx31_gripper_l_inner_joint1: axis 0 1 0 -> 0 0 -1; limit lower=0 upper=0.024 effort=500 velocity=1 -> lower=-0.7853981633974483 upper=0 effort=10 velocity=10; mimic (none) -> joint=idx41_gripper_l_outer_joint1 multiplier=-1 offset=0; origin xyz=-0.0265 0.0134 0.098 rpy=0 0 -1.5707969456925137 -> xyz=0 -0.0195 0.0565 rpy=-2.9951 -1.5707963267948966 -0.15964; type prismatic -> revolute
- joint idx41_gripper_l_outer_joint1: axis 0 1 0 -> 0 0 -1; limit lower=0 upper=0.024 effort=500 velocity=1 -> lower=0 upper=0.7853981633974483 effort=10 velocity=10; mimic joint=idx31_gripper_l_inner_joint1 multiplier=1 offset=0 -> (none); origin xyz=0.0265 -0.0134 0.098 rpy=0 0 1.5707969456925137 -> xyz=0 0.0195 0.0565 rpy=-2.9951 -1.5707963267948966 -0.15964; type prismatic -> revolute
- joint idx71_gripper_r_inner_joint1: axis 0 1 0 -> 0 0 -1; limit lower=0 upper=0.024 effort=500 velocity=1 -> lower=-0.7853981633974483 upper=0 effort=10 velocity=10; mimic (none) -> joint=idx81_gripper_r_outer_joint1 multiplier=-1 offset=0; origin xyz=-0.0265 0.0134 0.098 rpy=0 0 -1.5707969456925137 -> xyz=0 -0.0195 0.0565 rpy=-2.9951 -1.5707963267948966 -0.15964; type prismatic -> revolute
- joint idx81_gripper_r_outer_joint1: axis 0 1 0 -> 0 0 -1; limit lower=0 upper=0.024 effort=500 velocity=1 -> lower=0 upper=0.7853981633974483 effort=10 velocity=10; mimic joint=idx71_gripper_r_inner_joint1 multiplier=1 offset=0 -> (none); origin xyz=0.0265 -0.0134 0.098 rpy=0 0 1.5707969456925137 -> xyz=0 0.0195 0.0565 rpy=-2.9951 -1.5707963267948966 -0.15964; type prismatic -> revolute
