Commit message: rebuild adam_pick on 8e6f58b baseline with G1 gripper
Ultraworked with [Sisyphus](https://github.com/code-yeongyu/oh-my-openagent)

Co-authored-by: Sisyphus <clio-agent@sisyphuslabs.ai>

File: adam_pick/adam_pro_omnipicker.urdf (robot description, URDF)
Before this commit: robot adam_pro_omnipicker, 55 links, 54 joints
Links:
- removed link anklePitchLeft
- removed link anklePitchRight
- removed link elbowLeft
- removed link elbowRight
- removed link gripper_l_inner_link2
- removed link gripper_l_outer_link2
- removed link gripper_r_inner_link2
- removed link gripper_r_outer_link2
- removed link hipPitchLeft
- removed link hipPitchRight
- removed link hipRollLeft
- removed link hipRollRight
- removed link imu_link
- removed link left_zed_link
- removed link neckPitch_link
- removed link neckYaw_link
- removed link pelvis
- removed link right_zed_link
- removed link shinLeft
- removed link shinRight
- removed link shoulderPitchLeft
- removed link shoulderPitchRight
- removed link shoulderRollLeft
- removed link shoulderRollRight
- removed link shoulderYawLeft
- removed link shoulderYawRight
- removed link thighLeft
- removed link thighRight
- removed link toeLeft
- removed link toeRight
- removed link torso
- removed link waistPitch_link
- removed link waistRoll_link
- removed link wristPitchLeft
- removed link wristPitchRight
- removed link wristRollLeft
- removed link wristRollRight
- removed link wristYawLeft
- removed link wristYawRight
- added link arm_base_link
- added link arm_l_end_link, mass 0.06158; collision cylinder length=0.046 radius=0.0307999; visual cylinder length=0.046 radius=0.0307999
- added link arm_r_end_link, mass 0.06158; collision cylinder length=0.046 radius=0.0307999; visual cylinder length=0.046 radius=0.0307999
- added link genie; collision box size=0.2983398 0.3376392 1.; collision box size=0.5996094 0.449 0.3027344
- added link genie_arm_l_base_link, mass 0.37595; collision cylinder length=0.09135 radius=0.0542692; visual cylinder length=0.09135 radius=0.0542692
- added link genie_arm_l_link1, mass 0.4936; collision cylinder length=0.1664206 radius=0.0557927; visual cylinder length=0.1664206 radius=0.0557927
- added link genie_arm_l_link2, mass 0.46245; collision cylinder length=0.1808592 radius=0.0630242; visual cylinder length=0.1808592 radius=0.0630242
- added link genie_arm_l_link3, mass 0.50026; collision cylinder length=0.2206989 radius=0.0542326; visual cylinder length=0.2206989 radius=0.0542326
- added link genie_arm_l_link4, mass 0.27473; collision cylinder length=0.1549554 radius=0.0578917; visual cylinder length=0.1549554 radius=0.0578917
- added link genie_arm_l_link5, mass 0.25139; collision cylinder length=0.134524 radius=0.0456146; visual cylinder length=0.134524 radius=0.0456146
- added link genie_arm_l_link6, mass 0.26634; collision cylinder length=0.18166 radius=0.0485074; visual cylinder length=0.18166 radius=0.0485074
- added link genie_arm_r_base_link, mass 0.37595; collision cylinder length=0.09135 radius=0.0544722; visual cylinder length=0.09135 radius=0.0544722
- added link genie_arm_r_link1, mass 0.4936; collision cylinder length=0.1664272 radius=0.054839; visual cylinder length=0.1664272 radius=0.054839
- added link genie_arm_r_link2, mass 0.41662; collision cylinder length=0.1808592 radius=0.0630242; visual cylinder length=0.1808592 radius=0.0630242
- added link genie_arm_r_link3, mass 0.49413; collision cylinder length=0.220614 radius=0.0521616; visual cylinder length=0.220614 radius=0.0521616
- added link genie_arm_r_link4, mass 0.27473; collision cylinder length=0.1549554 radius=0.0578917; visual cylinder length=0.1549554 radius=0.0578917
- added link genie_arm_r_link5, mass 0.25139; collision cylinder length=0.1342381 radius=0.0456203; visual cylinder length=0.1342381 radius=0.0456203
- added link genie_arm_r_link6, mass 0.26634; collision cylinder length=0.1827249 radius=0.0485715; visual cylinder length=0.1827249 radius=0.0485715
- added link genie_body_link1, mass 3.2627544; collision box size=0.1606445 0.0555553 0.1328125; collision box size=0.1625977 0.0437565 0.1601562
- added link genie_body_link2, mass 7.531992; collision box size=0.3457031 0.1810772 0.3125; collision cylinder length=0.0869706 radius=0.0966232
- added link genie_head_link1, mass 0.4143429; visual mesh filename=meshes/genie_head_link1_visuals_head_link1_mesh.obj scale=1. 1. 1.
- added link genie_head_link2, mass 0.707064; collision sphere radius=0.1125707; visual mesh filename=meshes/genie_head_link2_visuals_head_link2_head_link2.obj scale=1. 1. 1.
- link gripper_l_base_link: geometry collision mesh filename=meshes/gripper_l_base_link_collisions_gripper_base_link_mes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 scale=1. 1. 1.; visual mesh filename=meshes/gripper_l_base_link_collisions_gripper_base_link_mes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 scale=1. 1. 1.
- link gripper_l_inner_link1: geometry collision mesh filename=meshes/gripper_l_inner_link1_collisions_inner_link1_mesh.obj scale=1. 1. 1.; visual mesh filename=meshes/gripper_l_inner_link1_collisions_inner_link1_mesh.obj scale=1. 1. 1.
- link gripper_l_inner_link3: geometry collision mesh filename=meshes/gripper_l_inner_link3_collisions_inner_link3_mesh.obj scale=1. 1. 1.; visual mesh filename=meshes/gripper_l_inner_link3_collisions_inner_link3_mesh.obj scale=1. 1. 1.
- link gripper_l_inner_link4: geometry collision mesh filename=meshes/gripper_l_inner_link4_collisions_inner_link4_mesh.obj scale=1. 1. 1.; visual mesh filename=meshes/gripper_l_inner_link4_collisions_inner_link4_mesh.obj scale=1. 1. 1.
- link gripper_l_outer_link1: geometry collision mesh filename=meshes/gripper_l_outer_link1_collisions_outer_link1_mesh.obj scale=1. 1. 1.; visual mesh filename=meshes/gripper_l_outer_link1_collisions_outer_link1_mesh.obj scale=1. 1. 1.
- link gripper_l_outer_link3: geometry collision mesh filename=meshes/gripper_l_outer_link3_collisions_outer_link3_mesh.obj scale=1. 1. 1.; visual mesh filename=meshes/gripper_l_outer_link3_collisions_outer_link3_mesh.obj scale=1. 1. 1.
- link gripper_l_outer_link4: geometry collision mesh filename=meshes/gripper_l_outer_link4_collisions_outer_link4_mesh.obj scale=1. 1. 1.; visual mesh filename=meshes/gripper_l_outer_link4_collisions_outer_link4_mesh.obj scale=1. 1. 1.
- link gripper_r_base_link: geometry collision mesh filename=meshes/gripper_r_base_link_collisions_gripper_base_link_mes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 scale=1. 1. 1.; visual mesh filename=meshes/gripper_r_base_link_collisions_gripper_base_link_mes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 scale=1. 1. 1.
- link gripper_r_inner_link1: geometry collision mesh filename=meshes/gripper_r_inner_link1_collisions_inner_link1_mesh.obj scale=1. 1. 1.; visual mesh filename=meshes/gripper_r_inner_link1_collisions_inner_link1_mesh.obj scale=1. 1. 1.
- link gripper_r_inner_link3: geometry collision mesh filename=meshes/gripper_r_inner_link3_collisions_inner_link3_mesh.obj scale=1. 1. 1.; visual mesh filename=meshes/gripper_r_inner_link3_collisions_inner_link3_mesh.obj scale=1. 1. 1.
- link gripper_r_inner_link4: geometry collision mesh filename=meshes/gripper_r_inner_link4_collisions_inner_link4_mesh.obj scale=1. 1. 1.; visual mesh filename=meshes/gripper_r_inner_link4_collisions_inner_link4_mesh.obj scale=1. 1. 1.
- link gripper_r_outer_link1: geometry collision mesh filename=meshes/gripper_r_outer_link1_collisions_outer_link1_mesh.obj scale=1. 1. 1.; visual mesh filename=meshes/gripper_r_outer_link1_collisions_outer_link1_mesh.obj scale=1. 1. 1.
- link gripper_r_outer_link3: geometry collision mesh filename=meshes/gripper_r_outer_link3_collisions_outer_link3_mesh.obj scale=1. 1. 1.; visual mesh filename=meshes/gripper_r_outer_link3_collisions_outer_link3_mesh.obj scale=1. 1. 1.
- link gripper_r_outer_link4: geometry collision mesh filename=meshes/gripper_r_outer_link4_collisions_outer_link4_mesh.obj scale=1. 1. 1.; visual mesh filename=meshes/gripper_r_outer_link4_collisions_outer_link4_mesh.obj scale=1. 1. 1.
Joints:
- removed joint anklePitch_Left
- removed joint anklePitch_Right
- removed joint ankleRoll_Left
- removed joint ankleRoll_Right
- removed joint elbow_Left
- removed joint elbow_Right
- removed joint hipPitch_Left
- removed joint hipPitch_Right
- removed joint hipRoll_Left
- removed joint hipRoll_Right
- removed joint hipYaw_Left
- removed joint hipYaw_Right
- removed joint idx39_gripper_l_inner_joint2
- removed joint idx49_gripper_l_outer_joint2
- removed joint idx79_gripper_r_inner_joint2
- removed joint idx89_gripper_r_outer_joint2
- removed joint imu_joint
- removed joint kneePitch_Left
- removed joint kneePitch_Right
- removed joint left_zed_joint
- removed joint neckPitch
- removed joint neckYaw
- removed joint right_zed_joint
- removed joint shoulderPitch_Left
- removed joint shoulderPitch_Right
- removed joint shoulderRoll_Left
- removed joint shoulderRoll_Right
- removed joint shoulderYaw_Left
- removed joint shoulderYaw_Right
- removed joint waistPitch
- removed joint waistRoll
- removed joint waistYaw
- removed joint wristPitch_Left
- removed joint wristPitch_Right
- removed joint wristRoll_Left
- removed joint wristRoll_Right
- removed joint wristYaw_Left
- removed joint wristYaw_Right
- added joint idx01_body_joint1: type prismatic, parent genie, child genie_body_link1, origin xyz=0. 0. 0.6485 rpy=0. 0. 0., axis 0. 0. 1., limit lower=0. upper=0.55 effort=100. velocity=0.1
- added joint idx02_body_joint2: type revolute, parent genie_body_link1, child genie_body_link2, origin xyz=0.131 0. 0.  rpy=-1.5707964 0. 0. , axis 0. 0. 1., limit lower=0. upper=1.5707963 effort=100. velocity=0.5
- added joint idx11_head_joint1: type revolute, parent genie_body_link2, child genie_head_link1, origin xyz=0. -0.441 0.  rpy=1.5707963 0. 0. , axis 0. 0. 1., limit lower=-1.5707963 upper=1.5707963 effort=50. velocity=0.9999999
- added joint idx12_head_joint2: type revolute, parent genie_head_link1, child genie_head_link2, origin xyz=0.050238 0. 0.060065 rpy=-1.5707963 0. 0. , axis 0. 0. 1., limit lower=-0.3490658 upper=0.5235988 effort=50. velocity=0.9999999
- added joint idx20_arm_base_joint: type fixed, parent genie_body_link2, child arm_base_link, origin xyz=0. -0.305 0.  rpy=1.5707963 0. 0. 
- added joint idx20_arm_l_base_joint: type fixed, parent arm_base_link, child genie_arm_l_base_link, origin xyz=0. 0.025 0.  rpy=-1.5707963 0. 0. 
- added joint idx21_arm_l_joint1: type revolute, parent genie_arm_l_base_link, child genie_arm_l_link1, origin xyz=0. 0. 0.1859 rpy=-0.0000002 0. 0. , axis 0. 0. 1., limit lower=-3.1399998 upper=3.1399998 effort=60. velocity=3.1399998
- added joint idx22_arm_l_joint2: type revolute, parent genie_arm_l_link1, child genie_arm_l_link2, origin xyz=0. 0. -0. rpy=-1.5707964 0. 1.5707964, axis 0. 0. 1., limit lower=-2.0899998 upper=2.0899998 effort=60. velocity=3.1399998
- added joint idx23_arm_l_joint3: type revolute, parent genie_arm_l_link2, child genie_arm_l_link3, origin xyz=-0.0000001 -0.305 0.  rpy=1.5707964 1.5707964 0. , axis 0. 0. 1., limit lower=-3.0999997 upper=3.0999997 effort=60. velocity=3.9249998
- added joint idx24_arm_l_joint4: type revolute, parent genie_arm_l_link3, child genie_arm_l_link4, origin xyz=0. 0. 0. rpy=-1.5707959 0. -3.1415925, axis 0. 0. 1., limit lower=-1.7499999 upper=1.4299999 effort=60. velocity=3.9249998
- added joint idx25_arm_l_joint5: type revolute, parent genie_arm_l_link4, child genie_arm_l_link5, origin xyz=0. -0.1975 0.0000001 rpy=-1.5707959 0. 3.1415925, axis 0. 0. 1., limit lower=-3.0999997 upper=3.0999997 effort=30. velocity=3.9249998
- added joint idx26_arm_l_joint6: type revolute, parent genie_arm_l_link5, child genie_arm_l_link6, origin xyz=0. -0. -0. rpy=-1.570797 0. 0. , axis 0. 0. 1., limit lower=-1.7399999 upper=1.7399999 effort=30. velocity=3.9249998
- added joint idx27_arm_l_joint7: type revolute, parent genie_arm_l_link6, child arm_l_end_link, origin xyz=0. -0.1805 -0.0000001 rpy=1.5707968 0. 0. , axis 0. 0. 1., limit lower=-3.0999997 upper=3.0999997 effort=30. velocity=3.9249998
- added joint idx60_arm_r_base_joint: type fixed, parent arm_base_link, child genie_arm_r_base_link, origin xyz=0. -0.025 -0.  rpy=-1.5707964 0. -3.1415925
- added joint idx61_arm_r_joint1: type revolute, parent genie_arm_r_base_link, child genie_arm_r_link1, origin xyz=0. 0. 0.188 rpy=0. 0. 0., axis 0. 0. 1., limit lower=-3.1399998 upper=3.1399998 effort=60. velocity=3.1399998
- added joint idx62_arm_r_joint2: type revolute, parent genie_arm_r_link1, child genie_arm_r_link2, origin xyz=0. 0. -0. rpy=-1.5707964 0. -1.5707964, axis 0. 0. 1., limit lower=-2.0899998 upper=2.0899998 effort=60. velocity=3.1399998
- added joint idx63_arm_r_joint3: type revolute, parent genie_arm_r_link2, child genie_arm_r_link3, origin xyz=0. -0.305 -0.  rpy=-1.6754674 -1.570796 -3.0369215, axis 0. 0. 1., limit lower=-3.0999997 upper=3.0999997 effort=60. velocity=3.9249998
- added joint idx64_arm_r_joint4: type revolute, parent genie_arm_r_link3, child genie_arm_r_link4, origin xyz=-0. 0. -0.0000002 rpy=-1.5707964 -0. 3.1415925, axis 0. 0. 1., limit lower=-1.4299999 upper=1.7499999 effort=60. velocity=3.9249998
- added joint idx65_arm_r_joint5: type revolute, parent genie_arm_r_link4, child genie_arm_r_link5, origin xyz=0.0000877 -0.1974999 0.0001863 rpy=-1.5698532 0.0009053 -3.1411479, axis 0. 0. 1., limit lower=-3.0999997 upper=3.0999997 effort=30. velocity=3.9249998
- added joint idx66_arm_r_joint6: type revolute, parent genie_arm_r_link5, child genie_arm_r_link6, origin xyz=0.0000879 0.0001862 -0.0000003 rpy=-1.5717394 0.0004441 -0.0009057, axis 0. 0. 1., limit lower=-1.7399999 upper=1.7399999 effort=30. velocity=3.9249998
- added joint idx67_arm_r_joint7: type revolute, parent genie_arm_r_link6, child arm_r_end_link, origin xyz=0. -0.1805 -0.  rpy=1.5707964 0. 0. , axis 0. 0. 1., limit lower=-3.0999997 upper=3.0999997 effort=30. velocity=3.9249998
- joint idx31_gripper_l_inner_joint1: axis 0 0 -1 -> 0. 0. 1.; limit lower=-0.7853981633974483 upper=0 effort=10 velocity=10 -> lower=-0.7853982 upper=0. effort=10. velocity=9.9999995; mimic joint=idx41_gripper_l_outer_joint1 multiplier=-1 offset=0 -> (none); origin xyz=0 -0.0195 0.0565 rpy=-2.9951 -1.5707963267948966 -0.15964 -> xyz=-0.0565 -0.0195 -0.  rpy=3.1284454 0.0000004 3.1415925
- joint idx32_gripper_l_inner_joint3: axis 0 0 -1 -> 0. 0. 1.; limit lower=-2 upper=2 effort=10 velocity=10 -> lower=-1.9999999 upper=1.9999999 effort=10. velocity=9.9999995; origin xyz=0.030852 0.018551 0 rpy=0 0 0 -> xyz=0.030852 -0.018551 -0.  rpy=3.1415925 -0.0000002 0.0000005
- joint idx33_gripper_l_inner_joint4: axis 0 0 1 -> 0. 0. 1.; limit lower=-2 upper=2 effort=10 velocity=10 -> lower=-1.9999999 upper=1.9999999 effort=10. velocity=9.9999995; origin xyz=0.018118 -0.01574 0 rpy=0 0 0 -> xyz=0.018118 -0.01574 -0.  rpy=0. -0. 0.0000007
- joint idx41_gripper_l_outer_joint1: axis 0 0 -1 -> 0. 0. 1.; limit lower=0 upper=0.7853981633974483 effort=10 velocity=10 -> lower=0. upper=0.7853982 effort=10. velocity=9.9999995; origin xyz=0 0.0195 0.0565 rpy=-2.9951 -1.5707963267948966 -0.15964 -> xyz=-0.0565 0.0195 -0.  rpy=3.1284454 0.0000004 3.1415925
- joint idx42_gripper_l_outer_joint3: axis 0 0 -1 -> 0. 0. 1.; limit lower=-2 upper=2 effort=10 velocity=10 -> lower=-1.9999999 upper=1.9999999 effort=10. velocity=9.9999995; origin xyz=0.030852 -0.018551 0 rpy=0 0 0 -> xyz=0.030852 0.018551 -0.  rpy=3.1415925 -0.0000002 0.0000005
- joint idx43_gripper_l_outer_joint4: axis 0 0 -1 -> 0. 0. 1.; limit lower=-2 upper=2 effort=10 velocity=10 -> lower=-1.9999999 upper=1.9999999 effort=10. velocity=9.9999995; origin xyz=0.018118 0.01574 0 rpy=0 0 0 -> xyz=0.018118 0.01574 0.  rpy=0. -0. 0.0000007
- joint idx51_ee_l_joint: axis 0 0 0 -> (none); origin xyz=0 0 0.0061 rpy=0 0 1.5707963267948966 -> xyz=-0. 0. 0. rpy=3.1415925 1.5707958 -1.5707964; parent arm_l_link7 -> arm_l_end_link
- joint idx52_gripper_l_center_joint: origin xyz=0.0 0.0 0.14308 rpy=0 0 -1.5707963267948966 -> xyz=-0.14308 0. -0.0000001 rpy=1.5707967 -0.0000002 -1.5707965
- joint idx71_gripper_r_inner_joint1: axis 0 0 -1 -> 0. 0. 1.; limit lower=-0.7853981633974483 upper=0 effort=10 velocity=10 -> lower=-0.7853982 upper=0. effort=10. velocity=9.9999995; mimic joint=idx81_gripper_r_outer_joint1 multiplier=-1 offset=0 -> (none); origin xyz=0 -0.0195 0.0565 rpy=-2.9951 -1.5707963267948966 -0.15964 -> xyz=-0.0565 -0.0195 -0.  rpy=3.1284454 0.0000002 -3.1415925
- joint idx72_gripper_r_inner_joint3: axis 0 0 -1 -> 0. 0. 1.; limit lower=-2 upper=2 effort=10 velocity=10 -> lower=-1.9999999 upper=1.9999999 effort=10. velocity=9.9999995; origin xyz=0.030852 0.018551 0 rpy=0 0 0 -> xyz=0.030852 -0.018551 0.  rpy=3.1415925 0.0000002 0.0000001
- joint idx73_gripper_r_inner_joint4: axis 0 0 1 -> 0. 0. 1.; limit lower=-2 upper=2 effort=10 velocity=10 -> lower=-1.9999999 upper=1.9999999 effort=10. velocity=9.9999995; origin xyz=0.018118 -0.01574 0 rpy=0 0 0 -> xyz=0.018118 -0.01574 -0.  rpy=-0. 0. -0.0000007
- joint idx81_gripper_r_outer_joint1: axis 0 0 -1 -> 0. 0. 1.; limit lower=0 upper=0.7853981633974483 effort=10 velocity=10 -> lower=0. upper=0.7853982 effort=10. velocity=9.9999995; origin xyz=0 0.0195 0.0565 rpy=-2.9951 -1.5707963267948966 -0.15964 -> xyz=-0.0565 0.0195 -0.  rpy=3.1284454 0.0000002 -3.1415925
- joint idx82_gripper_r_outer_joint3: axis 0 0 -1 -> 0. 0. 1.; limit lower=-2 upper=2 effort=10 velocity=10 -> lower=-1.9999999 upper=1.9999999 effort=10. velocity=9.9999995; origin xyz=0.030852 -0.018551 0 rpy=0 0 0 -> xyz=0.030852 0.018551 -0.  rpy=3.1415925 0.0000002 0.0000001
- joint idx83_gripper_r_outer_joint4: axis 0 0 -1 -> 0. 0. 1.; limit lower=-2 upper=2 effort=10 velocity=10 -> lower=-1.9999999 upper=1.9999999 effort=10. velocity=9.9999995; origin xyz=0.018118 0.01574 0 rpy=0 0 0 -> xyz=0.018118 0.01574 0.  rpy=-0. 0. -0.0000007
- joint idx91_ee_r_joint: axis 0 0 0 -> (none); origin xyz=0 0 0 rpy=0 0 -1.5707963267948966 -> xyz=-0. -0. -0.0000001 rpy=1.5707964 1.5707964 0. ; parent arm_r_link7 -> arm_r_end_link
- joint idx92_gripper_r_center_joint: origin xyz=0.0 0.0 0.14308 rpy=0 0 -1.5707963267948966 -> xyz=-0.14308 -0. -0.  rpy=1.5707965 -0.0000001 -1.5707961
