Commit message: limit G1 replacement to adam_pick gripper
Ultraworked with [Sisyphus](https://github.com/code-yeongyu/oh-my-openagent)

Co-authored-by: Sisyphus <clio-agent@sisyphuslabs.ai>

File: adam_pick/adam_pro_omnipicker.urdf (robot description, URDF)
Before this commit: robot robot, 38 links, 37 joints
Links:
- removed link arm_base_link
- removed link arm_l_end_link
- removed link arm_r_end_link
- removed link genie
- removed link genie_arm_l_base_link
- removed link genie_arm_l_link1
- removed link genie_arm_l_link2
- removed link genie_arm_l_link3
- removed link genie_arm_l_link4
- removed link genie_arm_l_link5
- removed link genie_arm_l_link6
- removed link genie_arm_r_base_link
- removed link genie_arm_r_link1
- removed link genie_arm_r_link2
- removed link genie_arm_r_link3
- removed link genie_arm_r_link4
- removed link genie_arm_r_link5
- removed link genie_arm_r_link6
- removed link genie_body_link1
- removed link genie_body_link2
- removed link genie_head_link1
- removed link genie_head_link2
- added link anklePitchLeft, mass 0.03014230; collision mesh filename=meshes_stl_0.25/anklePitchLeft.STL; visual mesh filename=meshes_stl_0.25/anklePitchLeft.STL
- added link anklePitchRight, mass 0.03014230; collision mesh filename=meshes_stl_0.25/anklePitchRight.STL; visual mesh filename=meshes_stl_0.25/anklePitchRight.STL
- added link elbowLeft, mass 0.91770702; collision mesh filename=meshes_stl_0.25/elbowLeft.STL; visual mesh filename=meshes_stl_0.25/elbowLeft.STL
- added link elbowRight, mass 0.91770702; collision mesh filename=meshes_stl_0.25/elbowRight.STL; visual mesh filename=meshes_stl_0.25/elbowRight.STL
- added link gripper_l_inner_link2, mass 0.022591
- added link gripper_l_outer_link2, mass 0.025142
- added link gripper_r_inner_link2, mass 0.022591
- added link gripper_r_outer_link2, mass 0.025142
- added link hipPitchLeft, mass 2.23379987; visual mesh filename=meshes_stl_0.25/hipPitchLeft.STL
- added link hipPitchRight, mass 2.23477271; visual mesh filename=meshes_stl_0.25/hipPitchRight.STL
- added link hipRollLeft, mass 1.35107789; collision mesh filename=meshes_stl_0.25/hipRollLeft.STL; visual mesh filename=meshes_stl_0.25/hipRollLeft.STL
- added link hipRollRight, mass 1.35169943; collision mesh filename=meshes_stl_0.25/hipRollRight.STL; visual mesh filename=meshes_stl_0.25/hipRollRight.STL
- added link imu_link
- added link left_zed_link
- added link neckPitch_link, mass 0.95620414; collision mesh filename=meshes_stl_0.25/neckPitch_link.STL; visual mesh filename=meshes_stl_0.25/neckPitch_link.STL
- added link neckYaw_link, mass 0.39916798; collision mesh filename=meshes_stl_0.25/neckYaw_link.STL; visual mesh filename=meshes_stl_0.25/neckYaw_link.STL
- added link pelvis, mass 10.35646604; collision mesh filename=meshes_stl_0.25/pelvis.STL; visual mesh filename=meshes_stl_0.25/pelvis.STL
- added link right_zed_link
- added link shinLeft, mass 2.25363003; collision mesh filename=meshes_stl_0.25/shinLeft.STL; visual mesh filename=meshes_stl_0.25/shinLeft.STL
- added link shinRight, mass 2.25459286; collision mesh filename=meshes_stl_0.25/shinRight.STL; visual mesh filename=meshes_stl_0.25/shinRight.STL
- added link shoulderPitchLeft, mass 0.21614811; collision mesh filename=meshes_stl_0.25/shoulderPitchLeft.STL; visual mesh filename=meshes_stl_0.25/shoulderPitchLeft.STL
- added link shoulderPitchRight, mass 0.21648747; collision mesh filename=meshes_stl_0.25/shoulderPitchRight.STL; visual mesh filename=meshes_stl_0.25/shoulderPitchRight.STL
- added link shoulderRollLeft, mass 1.07881773; collision mesh filename=meshes_stl_0.25/shoulderRollLeft.STL; visual mesh filename=meshes_stl_0.25/shoulderRollLeft.STL
- added link shoulderRollRight, mass 1.08875448; collision mesh filename=meshes_stl_0.25/shoulderRollRight.STL; visual mesh filename=meshes_stl_0.25/shoulderRollRight.STL
- added link shoulderYawLeft, mass 0.90142027; collision mesh filename=meshes_stl_0.25/shoulderYawLeft.STL; visual mesh filename=meshes_stl_0.25/shoulderYawLeft.STL
- added link shoulderYawRight, mass 0.90139273; collision mesh filename=meshes_stl_0.25/shoulderYawRight.STL; visual mesh filename=meshes_stl_0.25/shoulderYawRight.STL
- added link thighLeft, mass 6.43432841; collision mesh filename=meshes_stl_0.25/thighLeft.STL; visual mesh filename=meshes_stl_0.25/thighLeft.STL
- added link thighRight, mass 6.43084156; collision mesh filename=meshes_stl_0.25/thighRight.STL; visual mesh filename=meshes_stl_0.25/thighRight.STL
- added link toeLeft, mass 0.63479601; collision box size=0.24 0.1 0.02; visual mesh filename=meshes_stl_0.25/toeLeft.STL
- added link toeRight, mass 0.63480789; collision box size=0.24 0.1 0.02; visual mesh filename=meshes_stl_0.25/toeRight.STL
- added link torso, mass 12.73336771; collision mesh filename=meshes_stl_0.25/torso.STL; visual mesh filename=meshes_stl_0.25/torso.STL
- added link waistPitch_link, mass 0.56353777; collision mesh filename=meshes_stl_0.25/waistPitch_link.STL; visual mesh filename=meshes_stl_0.25/waistPitch_link.STL
- added link waistRoll_link, mass 2.36268465; visual mesh filename=meshes_stl_0.25/waistRoll_link.STL
- added link wristPitchLeft, mass 0.11963454; collision mesh filename=meshes_stl_0.25/wristPitchLeft.STL; visual mesh filename=meshes_stl_0.25/wristPitchLeft.STL
- added link wristPitchRight, mass 0.11963454; collision mesh filename=meshes_stl_0.25/wristPitchRight.STL; visual mesh filename=meshes_stl_0.25/wristPitchRight.STL
- added link wristRollLeft, mass 0.0421730312888237; visual mesh filename=meshes_stl_0.25/wristRoll.STL
- added link wristRollRight, mass 0.021808; visual mesh filename=meshes_stl_0.25/wristRoll.STL
- added link wristYawLeft, mass 0.95587869; collision mesh filename=meshes_stl_0.25/wristYawLeft.STL; visual mesh filename=meshes_stl_0.25/wristYawLeft.STL
- added link wristYawRight, mass 0.95587832; collision mesh filename=meshes_stl_0.25/wristYawRight.STL; visual mesh filename=meshes_stl_0.25/wristYawRight.STL
- link gripper_l_base_link: geometry collision mesh filename=assets/gripper_l_base_link_collisions_gripper_base_link_mes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; visual mesh filename=assets/gripper_l_base_link_visuals_gripper_base_link_mesh.o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
- link gripper_l_inner_link1: geometry collision mesh filename=assets/gripper_l_inner_link1_collisions_inner_link1_mesh.obj; visual mesh filename=assets/gripper_l_inner_link1_visuals_inner_link1_mesh.obj
- link gripper_l_inner_link3: geometry collision mesh filename=assets/gripper_l_inner_link3_collisions_inner_link3_mesh.obj; visual mesh filename=assets/gripper_l_inner_link3_visuals_inner_link3_mesh.obj
- link gripper_l_inner_link4: geometry collision mesh filename=assets/gripper_l_inner_link4_collisions_inner_link4_mesh.obj; visual mesh filename=assets/gripper_l_inner_link4_visuals_inner_link4_mesh.obj
- link gripper_l_outer_link1: geometry collision mesh filename=assets/gripper_l_outer_link1_collisions_outer_link1_mesh.obj; visual mesh filename=assets/gripper_l_outer_link1_visuals_outer_link1_mesh.obj
- link gripper_l_outer_link3: geometry collision mesh filename=assets/gripper_l_outer_link3_collisions_outer_link3_mesh.obj; visual mesh filename=assets/gripper_l_outer_link3_visuals_outer_link3_mesh.obj
- link gripper_l_outer_link4: geometry collision mesh filename=assets/gripper_l_outer_link4_collisions_outer_link4_mesh.obj; visual mesh filename=assets/gripper_l_outer_link4_visuals_outer_link4_mesh.obj
- link gripper_r_base_link: geometry collision mesh filename=assets/gripper_r_base_link_collisions_gripper_base_link_mes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; visual mesh filename=assets/gripper_r_base_link_visuals_gripper_base_link_mesh.o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
- link gripper_r_inner_link1: geometry collision mesh filename=assets/gripper_r_inner_link1_collisions_inner_link1_mesh.obj; visual mesh filename=assets/gripper_r_inner_link1_visuals_inner_link1_mesh.obj
- link gripper_r_inner_link3: geometry collision mesh filename=assets/gripper_r_inner_link3_collisions_inner_link3_mesh.obj; visual mesh filename=assets/gripper_r_inner_link3_visuals_inner_link3_mesh.obj
- link gripper_r_inner_link4: geometry collision mesh filename=assets/gripper_r_inner_link4_collisions_inner_link4_mesh.obj; visual mesh filename=assets/gripper_r_inner_link4_visuals_inner_link4_mesh.obj
- link gripper_r_outer_link1: geometry collision mesh filename=assets/gripper_r_outer_link1_collisions_outer_link1_mesh.obj; visual mesh filename=assets/gripper_r_outer_link1_visuals_outer_link1_mesh.obj
- link gripper_r_outer_link3: geometry collision mesh filename=assets/gripper_r_outer_link3_collisions_outer_link3_mesh.obj; visual mesh filename=assets/gripper_r_outer_link3_visuals_outer_link3_mesh.obj
- link gripper_r_outer_link4: geometry collision mesh filename=assets/gripper_r_outer_link4_collisions_outer_link4_mesh.obj; visual mesh filename=assets/gripper_r_outer_link4_visuals_outer_link4_mesh.obj
Joints:
- removed joint idx01_body_joint1
- removed joint idx02_body_joint2
- removed joint idx11_head_joint1
- removed joint idx12_head_joint2
- removed joint idx20_arm_base_joint
- removed joint idx20_arm_l_base_joint
- removed joint idx21_arm_l_joint1
- removed joint idx22_arm_l_joint2
- removed joint idx23_arm_l_joint3
- removed joint idx24_arm_l_joint4
- removed joint idx25_arm_l_joint5
- removed joint idx26_arm_l_joint6
- removed joint idx27_arm_l_joint7
- removed joint idx60_arm_r_base_joint
- removed joint idx61_arm_r_joint1
- removed joint idx62_arm_r_joint2
- removed joint idx63_arm_r_joint3
- removed joint idx64_arm_r_joint4
- removed joint idx65_arm_r_joint5
- removed joint idx66_arm_r_joint6
- removed joint idx67_arm_r_joint7
- added joint anklePitch_Left: type revolute, parent shinLeft, child anklePitchLeft, origin xyz=0 0 -0.36999999999995 rpy=0 0 0, axis 0 1 0, limit lower=-1.0 upper=0.35 effort=40 velocity=20
- added joint anklePitch_Right: type revolute, parent shinRight, child anklePitchRight, origin xyz=0 0 -0.369999999999911 rpy=0 0 0, axis 0 1 0, limit lower=-1.0 upper=0.35 effort=40 velocity=20
- added joint ankleRoll_Left: type revolute, parent anklePitchLeft, child toeLeft, origin xyz=0 0 0 rpy=0 0 0, axis 1 0 0, limit lower=-0.3491 upper=0.3491 effort=12 velocity=20
- added joint ankleRoll_Right: type revolute, parent anklePitchRight, child toeRight, origin xyz=0 0 0 rpy=0 0 0, axis 1 0 0, limit lower=-0.3491 upper=0.3491 effort=12 velocity=20
- added joint elbow_Left: type revolute, parent shoulderYawLeft, child elbowLeft, origin xyz=0 -0.0285000000009982 -0.182950000001738 rpy=0 0 0, axis 0 1 0, limit lower=-2.496 upper=0.209 effort=30 velocity=8
- added joint elbow_Right: type revolute, parent shoulderYawRight, child elbowRight, origin xyz=0 0.0284999999998828 -0.182950000001922 rpy=0 0 0, axis 0 1 0, limit lower=-2.496 upper=0.209 effort=30 velocity=8
- added joint hipPitch_Left: type revolute, parent pelvis, child hipPitchLeft, origin xyz=0 0.0961924921295064 -0.0332411879418571 rpy=-0.610865238197473 0 0, axis 0 1 0, limit lower=-2.164 upper=2.164 effort=230 velocity=15
- added joint hipPitch_Right: type revolute, parent pelvis, child hipPitchRight, origin xyz=0 -0.0961924781696877 -0.0332412045786055 rpy=0.610865238197555 0 0, axis 0 1 0, limit lower=-2.164 upper=2.164 effort=230 velocity=15
- added joint hipRoll_Left: type revolute, parent hipPitchLeft, child hipRollLeft, origin xyz=-0.0254999999999983 0.0690000000000026 0 rpy=0.610865238197473 0 0, axis 1 0 0, limit lower=-0.733 upper=1.605 effort=160 velocity=8
- added joint hipRoll_Right: type revolute, parent hipPitchRight, child hipRollRight, origin xyz=-0.0254999999999981 -0.0689999999999357 0 rpy=-0.610865238197555 0 0, axis 1 0 0, limit lower=-1.605 upper=0.733 effort=160 velocity=8
- added joint hipYaw_Left: type revolute, parent hipRollLeft, child thighLeft, origin xyz=0.0440000071360198 0 -0.0524999940193389 rpy=0 0 0, axis 0 0 1, limit lower=-0.785 upper=0.785 effort=105 velocity=8
- added joint hipYaw_Right: type revolute, parent hipRollRight, child thighRight, origin xyz=0.0439999724402559 0 -0.0525000230976866 rpy=0 0 0, axis 0 0 1, limit lower=-0.785 upper=0.785 effort=105 velocity=8
- added joint idx39_gripper_l_inner_joint2: type revolute, parent gripper_l_base_link, child gripper_l_inner_link2, origin xyz=0 -0.021633 0.07387 rpy=-2.9951 -1.5707963267948966 -0.15964, axis 0 0 -1, limit lower=-2 upper=2 effort=10 velocity=10
- added joint idx49_gripper_l_outer_joint2: type revolute, parent gripper_l_base_link, child gripper_l_outer_link2, origin xyz=0 0.021633 0.07387 rpy=-2.9951 -1.5707963267948966 -0.15964, axis 0 0 -1, limit lower=-2 upper=2 effort=10 velocity=10
- added joint idx79_gripper_r_inner_joint2: type revolute, parent gripper_r_base_link, child gripper_r_inner_link2, origin xyz=0 -0.021633 0.07387 rpy=-2.9951 -1.5707963267948966 -0.15964, axis 0 0 -1, limit lower=-2 upper=2 effort=10 velocity=10
- added joint idx89_gripper_r_outer_joint2: type revolute, parent gripper_r_base_link, child gripper_r_outer_link2, origin xyz=0 0.021633 0.07387 rpy=-2.9951 -1.5707963267948966 -0.15964, axis 0 0 -1, limit lower=-2 upper=2 effort=10 velocity=10
- added joint imu_joint: type fixed, parent pelvis, child imu_link, origin xyz=0 0 0 rpy=0 0 0
- added joint kneePitch_Left: type revolute, parent thighLeft, child shinLeft, origin xyz=0 -0.0354999999998497 -0.369000000000099 rpy=0 0 0, axis 0 1 0, limit lower=0.052 upper=2.391 effort=230 velocity=15
- added joint kneePitch_Right: type revolute, parent thighRight, child shinRight, origin xyz=0 0.0354999999997395 -0.368999999999986 rpy=0 0 0, axis 0 1 0, limit lower=0.052 upper=2.391 effort=230 velocity=15
- added joint left_zed_joint: type fixed, parent neckPitch_link, child left_zed_link, origin xyz=0.096 0.0118 0.0407 rpy=0 0 0
- added joint neckPitch: type revolute, parent neckYaw_link, child neckPitch_link, origin xyz=0.0316000000000086 0.0199499999999967 0.145949999999989 rpy=0 0 0, axis 0 1 0, limit lower=-0.873 upper=0.873 effort=6.4 velocity=5
- added joint neckYaw: type revolute, parent torso, child neckYaw_link, origin xyz=-0.0130000000000059 0 0.298550000000013 rpy=0 0 0, axis 0 0 1, limit lower=-1.571 upper=1.571 effort=6.4 velocity=5
- added joint right_zed_joint: type fixed, parent neckPitch_link, child right_zed_link, origin xyz=0.096 -0.0517 0.0407 rpy=0 0 0
- added joint shoulderPitch_Left: type revolute, parent torso, child shoulderPitchLeft, origin xyz=0 0.165093970689425 0.259229560594865 rpy=0.349065850393456 0 0, axis 0 1 0, limit lower=-3.613 upper=2.042 effort=65 velocity=8
- added joint shoulderPitch_Right: type revolute, parent torso, child shoulderPitchRight, origin xyz=0 -0.165093970689321 0.259229560595242 rpy=-0.349065850398898 0 0, axis 0 1 0, limit lower=-3.613 upper=2.042 effort=65 velocity=8
- added joint shoulderRoll_Left: type revolute, parent shoulderPitchLeft, child shoulderRollLeft, origin xyz=0.036199999996826 0.0434999999975074 0 rpy=-0.349065850393456 0 0, axis 1 0 0, limit lower=-0.628 upper=2.793 effort=65 velocity=8
- added joint shoulderRoll_Right: type revolute, parent shoulderPitchRight, child shoulderRollRight, origin xyz=0.036199999639011 -0.0435000000171988 0 rpy=0.349065850398898 0 0, axis 1 0 0, limit lower=-2.793 upper=0.628 effort=65 velocity=8
- added joint shoulderYaw_Left: type revolute, parent shoulderRollLeft, child shoulderYawLeft, origin xyz=-0.0361999999622004 0.0340000000110588 -0.0796999999903454 rpy=0 0 0, axis 0 0 1, limit lower=-2.583 upper=2.583 effort=65 velocity=8
- added joint shoulderYaw_Right: type revolute, parent shoulderRollRight, child shoulderYawRight, origin xyz=-0.0361999996389017 -0.0339999999996759 -0.0797000000498751 rpy=0 0 0, axis 0 0 1, limit lower=-2.583 upper=2.583 effort=65 velocity=8
- added joint waistPitch: type revolute, parent waistRoll_link, child waistPitch_link, origin xyz=0 0 0.08 rpy=0 0 0, axis 0 1 0, limit lower=-0.663 upper=1.361 effort=110 velocity=8
- added joint waistRoll: type revolute, parent pelvis, child waistRoll_link, origin xyz=0 0 0.0440000000007929 rpy=0 0 0, axis 1 0 0, limit lower=-0.279 upper=0.279 effort=110 velocity=8
- added joint waistYaw: type revolute, parent waistPitch_link, child torso, origin xyz=0 0.000500000000007081 0.05299999999999 rpy=0 0 0, axis 0 0 1, limit lower=-0.829 upper=0.829 effort=110 velocity=8
- added joint wristPitch_Left: type revolute, parent wristYawLeft, child wristPitchLeft, origin xyz=0 0 -0.201699999999994 rpy=0 0 0, axis 0 1 0, limit lower=-0.96 upper=0.96 effort=6.4 velocity=5
- added joint wristPitch_Right: type revolute, parent wristYawRight, child wristPitchRight, origin xyz=0 0 -0.201699999999861 rpy=0 0 0, axis 0 1 0, limit lower=-0.96 upper=0.96 effort=6.4 velocity=5
- added joint wristRoll_Left: type revolute, parent wristPitchLeft, child wristRollLeft, origin xyz=0 0 0 rpy=0 0 0, axis 1 0 0, limit lower=-0.907 upper=0.907 effort=6.4 velocity=4.9218
- added joint wristRoll_Right: type revolute, parent wristPitchRight, child wristRollRight, origin xyz=0 0 0 rpy=0 0 0, axis 1 0 0, limit lower=-0.907 upper=0.907 effort=6.4 velocity=4.9218
- added joint wristYaw_Left: type revolute, parent elbowLeft, child wristYawLeft, origin xyz=-0.0250000000083053 0.028499999997574 -0.0728999999980683 rpy=0 0 0, axis 0 0 1, limit lower=-2.67 upper=2.67 effort=6.4 velocity=5
- added joint wristYaw_Right: type revolute, parent elbowRight, child wristYawRight, origin xyz=-0.0249999999999065 -0.0285000000002922 -0.0728999999999894 rpy=0 0 0, axis 0 0 1, limit lower=-2.67 upper=2.67 effort=6.4 velocity=5
- joint idx31_gripper_l_inner_joint1: axis 0. 0. 1. -> 0 0 -1; limit lower=-0.7853982 upper=0. effort=10. velocity=9.9999995 -> lower=-0.7853981633974483 upper=0 effort=10 velocity=10; mimic (none) -> joint=idx41_gripper_l_outer_joint1 multiplier=-1 offset=0; origin xyz=-0.0565 -0.0195 -0.  rpy=3.1284454 0.0000004 3.1415925 -> xyz=0 -0.0195 0.0565 rpy=-2.9951 -1.5707963267948966 -0.15964
- joint idx32_gripper_l_inner_joint3: axis 0. 0. 1. -> 0 0 -1; limit lower=-1.9999999 upper=1.9999999 effort=10. velocity=9.9999995 -> lower=-2 upper=2 effort=10 velocity=10; origin xyz=0.030852 -0.018551 -0.  rpy=3.1415925 -0.0000002 0.0000005 -> xyz=0.030852 0.018551 0 rpy=0 0 0
- joint idx33_gripper_l_inner_joint4: axis 0. 0. 1. -> 0 0 1; limit lower=-1.9999999 upper=1.9999999 effort=10. velocity=9.9999995 -> lower=-2 upper=2 effort=10 velocity=10; origin xyz=0.018118 -0.01574 -0.  rpy=0. -0. 0.0000007 -> xyz=0.018118 -0.01574 0 rpy=0 0 0
- joint idx41_gripper_l_outer_joint1: axis 0. 0. 1. -> 0 0 -1; limit lower=0. upper=0.7853982 effort=10. velocity=9.9999995 -> lower=0 upper=0.7853981633974483 effort=10 velocity=10; origin xyz=-0.0565 0.0195 -0.  rpy=3.1284454 0.0000004 3.1415925 -> xyz=0 0.0195 0.0565 rpy=-2.9951 -1.5707963267948966 -0.15964
- joint idx42_gripper_l_outer_joint3: axis 0. 0. 1. -> 0 0 -1; limit lower=-1.9999999 upper=1.9999999 effort=10. velocity=9.9999995 -> lower=-2 upper=2 effort=10 velocity=10; origin xyz=0.030852 0.018551 -0.  rpy=3.1415925 -0.0000002 0.0000005 -> xyz=0.030852 -0.018551 0 rpy=0 0 0
- joint idx43_gripper_l_outer_joint4: axis 0. 0. 1. -> 0 0 -1; limit lower=-1.9999999 upper=1.9999999 effort=10. velocity=9.9999995 -> lower=-2 upper=2 effort=10 velocity=10; origin xyz=0.018118 0.01574 0.  rpy=0. -0. 0.0000007 -> xyz=0.018118 0.01574 0 rpy=0 0 0
- joint idx51_ee_l_joint: axis (none) -> 0 0 0; origin xyz=-0. 0. 0. rpy=3.1415925 1.5707958 -1.5707964 -> xyz=0 0 0 rpy=0 0 1.5707963267948966; parent arm_l_end_link -> wristRollLeft
- joint idx52_gripper_l_center_joint: origin xyz=-0.14308 0. -0.0000001 rpy=1.5707967 -0.0000002 -1.5707965 -> xyz=0.0 0.0 0.14308 rpy=0 0 -1.5707963267948966
- joint idx71_gripper_r_inner_joint1: axis 0. 0. 1. -> 0 0 -1; limit lower=-0.7853982 upper=0. effort=10. velocity=9.9999995 -> lower=-0.7853981633974483 upper=0 effort=10 velocity=10; mimic (none) -> joint=idx81_gripper_r_outer_joint1 multiplier=-1 offset=0; origin xyz=-0.0565 -0.0195 -0.  rpy=3.1284454 0.0000002 -3.1415925 -> xyz=0 -0.0195 0.0565 rpy=-2.9951 -1.5707963267948966 -0.15964
- joint idx72_gripper_r_inner_joint3: axis 0. 0. 1. -> 0 0 -1; limit lower=-1.9999999 upper=1.9999999 effort=10. velocity=9.9999995 -> lower=-2 upper=2 effort=10 velocity=10; origin xyz=0.030852 -0.018551 0.  rpy=3.1415925 0.0000002 0.0000001 -> xyz=0.030852 0.018551 0 rpy=0 0 0
- joint idx73_gripper_r_inner_joint4: axis 0. 0. 1. -> 0 0 1; limit lower=-1.9999999 upper=1.9999999 effort=10. velocity=9.9999995 -> lower=-2 upper=2 effort=10 velocity=10; origin xyz=0.018118 -0.01574 -0.  rpy=-0. 0. -0.0000007 -> xyz=0.018118 -0.01574 0 rpy=0 0 0
- joint idx81_gripper_r_outer_joint1: axis 0. 0. 1. -> 0 0 -1; limit lower=0. upper=0.7853982 effort=10. velocity=9.9999995 -> lower=0 upper=0.7853981633974483 effort=10 velocity=10; origin xyz=-0.0565 0.0195 -0.  rpy=3.1284454 0.0000002 -3.1415925 -> xyz=0 0.0195 0.0565 rpy=-2.9951 -1.5707963267948966 -0.15964
- joint idx82_gripper_r_outer_joint3: axis 0. 0. 1. -> 0 0 -1; limit lower=-1.9999999 upper=1.9999999 effort=10. velocity=9.9999995 -> lower=-2 upper=2 effort=10 velocity=10; origin xyz=0.030852 0.018551 -0.  rpy=3.1415925 0.0000002 0.0000001 -> xyz=0.030852 -0.018551 0 rpy=0 0 0
- joint idx83_gripper_r_outer_joint4: axis 0. 0. 1. -> 0 0 1; limit lower=-1.9999999 upper=1.9999999 effort=10. velocity=9.9999995 -> lower=-2 upper=2 effort=10 velocity=10; origin xyz=0.018118 0.01574 0.  rpy=-0. 0. -0.0000007 -> xyz=0.018118 0.01574 0 rpy=0 0 0
- joint idx91_ee_r_joint: axis (none) -> 0 0 0; origin xyz=-0. -0. -0.0000001 rpy=1.5707964 1.5707964 0.  -> xyz=0 0 0 rpy=0 0 -1.5707963267948966; parent arm_r_end_link -> wristRollRight
- joint idx92_gripper_r_center_joint: origin xyz=-0.14308 -0. -0.  rpy=1.5707965 -0.0000001 -1.5707961 -> xyz=0.0 0.0 0.14308 rpy=0 0 -1.5707963267948966

Commit message: adjust link1 mesh-only orientation in adam_pick gripper
Ultraworked with [Sisyphus](https://github.com/code-yeongyu/oh-my-openagent)

Co-authored-by: Sisyphus <clio-agent@sisyphuslabs.ai>

File: adam_pick/adam_pro_omnipicker.urdf (robot description, URDF)
Before this commit: robot adam_pro_omnipicker, 55 links, 54 joints
Joints:
- joint idx51_ee_l_joint: origin xyz=0 0 0 rpy=0 0 1.5707963267948966 -> xyz=0 0 -0.049 rpy=0 3.14 0
- joint idx91_ee_r_joint: origin xyz=0 0 0 rpy=0 0 -1.5707963267948966 -> xyz=0 0 -0.049 rpy=3.14 0 0
