Commit message: updateadampro

File: adam_pro/adam_pro.urdf (robot description, URDF)
Before this commit: robot adam_pro, 57 links, 56 joints
Joints:
- joint L_index_DIP_joint: axis (none) -> -1 0 0; limit (none) -> lower=0 upper=1.6 effort=1 velocity=1; mimic (none) -> joint=L_index_MCP_joint multiplier=1 offset=0; type fixed -> revolute
- joint L_index_MCP_joint: axis (none) -> -1 0 0; limit (none) -> lower=0 upper=1.7 effort=1 velocity=1; type fixed -> revolute
- joint L_middle_DIP_joint: axis (none) -> -1 0 0; limit (none) -> lower=0 upper=1.6 effort=1 velocity=1; mimic (none) -> joint=L_middle_MCP_joint multiplier=1 offset=0; type fixed -> revolute
- joint L_middle_MCP_joint: axis (none) -> -1 0 0; limit (none) -> lower=0 upper=1.7 effort=1 velocity=1; type fixed -> revolute
- joint L_pinky_DIP_joint: axis (none) -> -1 0 0; limit (none) -> lower=0 upper=1.6 effort=1 velocity=1; mimic (none) -> joint=L_pinky_MCP_joint multiplier=1 offset=0; type fixed -> revolute
- joint L_pinky_MCP_joint: axis (none) -> -1 0 0; limit (none) -> lower=0 upper=1.7 effort=1 velocity=1; type fixed -> revolute
- joint L_ring_DIP_joint: axis (none) -> -1 0 0; limit (none) -> lower=0 upper=1.6 effort=1 velocity=1; mimic (none) -> joint=L_ring_MCP_joint multiplier=1 offset=0; type fixed -> revolute
- joint L_ring_MCP_joint: axis (none) -> -1 0 0; limit (none) -> lower=0 upper=1.7 effort=1 velocity=1; type fixed -> revolute
- joint L_thumb_DIP_joint: axis (none) -> 0 1 0; limit (none) -> lower=0 upper=1.2 effort=1 velocity=1; mimic (none) -> joint=L_thumb_MCP_joint2 multiplier=2.4 offset=0; type fixed -> revolute
- joint L_thumb_MCP_joint1: axis (none) -> 0 0 -1; limit (none) -> lower=0 upper=1.1 effort=1 velocity=1; type fixed -> revolute
- joint L_thumb_MCP_joint2: axis (none) -> 0 1 0; limit (none) -> lower=0 upper=0.5 effort=1 velocity=1; type fixed -> revolute
- joint L_thumb_PIP_joint: axis (none) -> 0 1 0; limit (none) -> lower=0 upper=1 effort=1 velocity=1; mimic (none) -> joint=L_thumb_MCP_joint2 multiplier=1.6 offset=0; type fixed -> revolute
- joint R_index_DIP_joint: axis (none) -> 1 0 0; limit (none) -> lower=0 upper=1.6 effort=1 velocity=1; mimic (none) -> joint=R_index_MCP_joint multiplier=1 offset=0; type fixed -> revolute
- joint R_index_MCP_joint: axis (none) -> 1 0 0; limit (none) -> lower=0 upper=1.7 effort=1 velocity=1; type fixed -> revolute
- joint R_middle_DIP_joint: axis (none) -> 1 0 0; limit (none) -> lower=0 upper=1.6 effort=1 velocity=1; mimic (none) -> joint=R_middle_MCP_joint multiplier=1 offset=0; type fixed -> revolute
- joint R_middle_MCP_joint: axis (none) -> 1 0 0; limit (none) -> lower=0 upper=1.7 effort=1 velocity=1; type fixed -> revolute
- joint R_pinky_DIP_joint: axis (none) -> 1 0 0; limit (none) -> lower=0 upper=1.6 effort=1 velocity=1; mimic (none) -> joint=R_pinky_MCP_joint multiplier=1 offset=0; type fixed -> revolute
- joint R_pinky_MCP_joint: axis (none) -> 1 0 0; limit (none) -> lower=0 upper=1.7 effort=1 velocity=1; type fixed -> revolute
- joint R_ring_DIP_joint: axis (none) -> 1 0 0; limit (none) -> lower=0 upper=1.6 effort=1 velocity=1; mimic (none) -> joint=R_ring_MCP_joint multiplier=1 offset=0; type fixed -> revolute
- joint R_ring_MCP_joint: axis (none) -> 1 0 0; limit (none) -> lower=0 upper=1.7 effort=1 velocity=1; type fixed -> revolute
- joint R_thumb_DIP_joint: axis (none) -> 0 1 0; limit (none) -> lower=0 upper=1.2 effort=1 velocity=1; mimic (none) -> joint=R_thumb_MCP_joint2 multiplier=2.4 offset=0; type fixed -> revolute
- joint R_thumb_MCP_joint1: axis (none) -> 0 0 1; limit (none) -> lower=0 upper=1.1 effort=1 velocity=1; type fixed -> revolute
- joint R_thumb_MCP_joint2: axis (none) -> 0 1 0; limit (none) -> lower=0 upper=0.5 effort=1 velocity=1; type fixed -> revolute
- joint R_thumb_PIP_joint: axis (none) -> 0 1 0; limit (none) -> lower=0 upper=1 effort=1 velocity=1; mimic (none) -> joint=R_thumb_MCP_joint2 multiplier=1.6 offset=0; type fixed -> revolute
- joint neckPitch: axis (none) -> 0 1 0; limit (none) -> lower=-0.873 upper=0.873 effort=6.4 velocity=5; type fixed -> revolute
- joint neckYaw: axis (none) -> 0 0 1; limit (none) -> lower=-1.571 upper=1.571 effort=6.4 velocity=5; type fixed -> revolute
- joint wristPitch_Left: axis (none) -> 0 1 0; limit (none) -> lower=-0.96 upper=0.96 effort=6.4 velocity=5; type fixed -> revolute
- joint wristPitch_Right: axis (none) -> 0 1 0; limit (none) -> lower=-0.96 upper=0.96 effort=6.4 velocity=5; type fixed -> revolute
- joint wristRoll_Left: axis (none) -> 1 0 0; limit (none) -> lower=-0.96 upper=0.96 effort=6.4 velocity=5; type fixed -> revolute
- joint wristRoll_Right: axis (none) -> 1 0 0; limit (none) -> lower=-0.96 upper=0.96 effort=6.4 velocity=5; type fixed -> revolute
- joint wristYaw_Left: axis (none) -> 0 0 1; limit (none) -> lower=-2.67 upper=2.67 effort=6.4 velocity=5; type fixed -> revolute
- joint wristYaw_Right: axis (none) -> 0 0 1; limit (none) -> lower=-2.67 upper=2.67 effort=6.4 velocity=5; type fixed -> revolute
